File: relay_board.brd (EAGLE design)
At the start: 37 x 67 mm, 21 parts, among them IC1 REG1117, K1 JS-M1-9V-4

Commit message: Eh
Parts:
- removed K1: JS-M1-9V-4, relay:JS-M
- removed Q1: (no value), SparkFun-DiscreteSemi:SOT223
- removed U$2: HLK-PM03, PowerSocket:HLK-PM03
- added B1: DBS104G, rectifier:DBS
- added C10: 100uf 16V, SparkFun-Capacitors:CPOL-RADIAL-100UF-25V
- added C3: 0.1uf, SparkFun-Capacitors:0805
- added C4: 10000pf/400V, resistor:C050-045X075
- added C5: 50000pf/400V, resistor:C150-072X183
- added C6, C7: 4.7uf, rcl:E3,5-10
- added C8: 0.1uf, SparkFun-Capacitors:CAP-PTH-SMALL-KIT
- added C9: 10uf 35V, SparkFun-Capacitors:CPOL-RADIAL-10UF-25V-KIT
- added D1: 1N4005GP, diode:DO41-10
- added D2: BYV26C, diode:SOD57-10
- added DA1: (no value), lnk306:LNK306_SMB
- added L1: SLF7045, inductors:SLF7045
- added L2: (no value), SparkFun-Passives:DR1030
- added R10: 470, SparkFun-Resistors:AXIAL-0.4
- added R11: 360, SparkFun-Resistors:AXIAL-0.4
- added R12: 8.2Ohm, SparkFun-Resistors:AXIAL-0.6
- added R13: (no value), rcl:M0805
- added R14: 2.05k 1%, SparkFun-Resistors:0805
- added R15: 3.84k 1%, SparkFun-Resistors:0805
- added R16: 3.3k, rcl:M0805
- added R9: 39Ohm/1W, SparkFun-Resistors:AXIAL-0.6
- added T1: BT136, triac:TO220AB
- added U1: (no value), SparkFun-DiscreteSemi:DIP8SMD
- R1, R2, R3, R4: device SparkFun-Resistors:0805 -> rcl:M0805
- moved R6 96.3 mm to (99.1, 2.06)
- moved R4 91.3 mm to (104.9, 40.6)
- moved S1 87.1 mm to (105.2, 40.4)
- moved R5 83.9 mm to (95.7, 27.0)
- moved J1 83.7 mm to (84.0, 10.6)
- moved U$1 81.0 mm to (111.0, 6.75)
- moved R8 79.5 mm to (108.1, 27.1)
- moved R7 79.1 mm to (103.5, 27.0)
- moved C1 77.9 mm to (110.8, 2.06)
- moved LED1 68.1 mm to (86.3, 56.0)
- moved C2 67.5 mm to (-47.6, 56.0)
- moved R2 60.4 mm to (76.8, 57.7)
- moved R3 60.3 mm to (80.8, 56.8)
- moved IC1 60.3 mm to (-49.4, 54.8)
- moved R1 60.2 mm to (78.7, 57.6)
Connections:
- new net N$10: B1.-, C6.+, L1.1
- new net N$12: R13.1, U1.1
- new net N$13: C8.2, C9.2, D2.C, DA1.1, L2.1, R14.1
- new net N$14: C8.1, DA1.3
- new net N$15: DA1.4, R14.2, R15.1
- new net N$16: C9.1, D1.C, R15.2
- new net N$5: C4.1, R9.P$1
- new net N$6: C5.1, R10.P$1, R11.P$2
- new net N$7: T1.3, U1.4
- new net N$8: C7.+, DA1.5, L1.2
- new net N$9: B1.AC2, R12.P$2
- net 3.3V: now also C3.1
- net 5V: now also C10.1, D1.A, L2.2, R16.2; no longer Q1.2, U$2.+VO
- net GND: now also B1.+, C10.2, C3.2, C6.-, C7.-, D2.A, R16.1, U1.2; no longer K1.2, U$2.-VO
- net LIVE_IN: now also R10.P$2, R12.P$1, R9.P$2, T1.1; no longer K1.C, U$2.AC1
- net LIVE_OUT: now also C4.2, C5.2, T1.2; no longer K1.NO
- net N$4: now also R11.P$1, U1.6; no longer K1.1, Q1.3
- net NEUTRAL: now also B1.AC1; no longer U$2.AC2
- net RELAY: now also R13.2; no longer Q1.1
Routing:
- net 3.3V: track 118.3 -> 0.00 mm
- net 5V: track 56.2 -> 0.00 mm, vias 1 -> 0
- net BLUE: track 45.6 -> 0.00 mm, vias 2 -> 0
- net GREEN: track 45.1 -> 0.00 mm, vias 2 -> 0
- net RED: track 45.1 -> 0.00 mm, vias 2 -> 0
- net LIVE_IN: track 72.1 -> 27.2 mm
- net RELAY: track 27.6 -> 0.00 mm
- net RESET: track 25.4 -> 0.00 mm
- net CH_PD: track 23.6 -> 0.00 mm
- net RX: track 23.5 -> 0.00 mm
- net TX: track 21.8 -> 0.00 mm
- net N$6: track 0.00 -> 21.0 mm
- net NEUTRAL: track 13.1 -> 32.6 mm
- net LIVE_OUT: track 56.2 -> 40.8 mm
- net N$7: track 0.00 -> 15.2 mm
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- added copper zone on layer 16, net LIVE_IN
- added copper zone on layer 1, net LIVE_OUT
Other:
- board text removed: "3.3v"
- board text removed: "gnd"
- board text removed: "rx"
- board text removed: "tx"
