File: relay_board.sch (EAGLE design)
At the start: 21 parts, among them IC1 REG1117, K1 JS-M1-9V-4

Commit message: Eh
Parts:
- removed K1: JS-M1-9V-4, relay:JS-M1-9V-4
- removed Q1: (no value), SparkFun-DiscreteSemi:TRANSISTOR_NPNSMD2
- removed U$2: HLK-PM03, PowerSocket:HLK-PM03
- added B1: DBS104G, rectifier:DBS104G
- added C10: 100uf 16V, SparkFun-Capacitors:100UF-25V-20%(PTH)
- added C3: 0.1uf, SparkFun-Capacitors:CAP0805
- added C4: 10000pf/400V, resistor:C-EU050-045X075
- added C5: 50000pf/400V, resistor:C-EU150-072X183
- added C6, C7: 4.7uf, rcl:CPOL-EUE3.5-10
- added C8: 0.1uf, SparkFun-Capacitors:0.1UF-50V-20%(PTH)KIT-EZ
- added C9: 10uf 35V, SparkFun-Capacitors:10UF-25V-20%(PTH)KIT
- added D1: 1N4005GP, diode:1N4004
- added D2: BYV26C, diode:BYV27
- added DA1: (no value), lnk306:LNK306LNK306
- added L1: SLF7045, inductors:SLF7045
- added L2: (no value), SparkFun-Passives:INDUCTORDR1030
- added R10: 470, SparkFun-Resistors:RESISTORPTH-1/4W
- added R11: 360, SparkFun-Resistors:RESISTORPTH-1/4W
- added R12: 8.2Ohm, SparkFun-Resistors:RESISTORPTH-1W
- added R13: (no value), rcl:R-EU_M0805
- added R14: 2.05k 1%, SparkFun-Resistors:RESISTOR0805-RES
- added R15: 3.84k 1%, SparkFun-Resistors:RESISTOR0805-RES
- added R16: 3.3k, rcl:R-EU_M0805
- added R9: 39Ohm/1W, SparkFun-Resistors:RESISTORPTH-1W
- added T1: BT136, triac:BT136
- added U1: (no value), SparkFun-DiscreteSemi:MOC3063S
- R1, R2, R3, R4: device SparkFun-Resistors:RESISTOR0805-RES -> rcl:R-EU_M0805
Connections:
- new net N$10: B1.-, C6.+, L1.1
- new net N$12: R13.1, U1.A
- new net N$13: C8.2, C9.-, D2.C, DA1.S, L2.1, R14.1
- new net N$14: C8.1, DA1.BP
- new net N$15: DA1.FB, R14.2, R15.1
- new net N$16: C9.+, D1.C, R15.2
- new net N$5: C4.1, R9.1
- new net N$6: C5.1, R10.1, R11.2
- new net N$7: T1.G, U1.T2
- new net N$8: C7.+, DA1.D, L1.2
- new net N$9: B1.AC2, R12.2
- net 3.3V: now also C3.1
- net 5V: now also C10.+, D1.A, L2.2, R16.2; no longer Q1.C, U$2.+VO
- net GND: now also B1.+, C10.-, C3.2, C6.-, C7.-, D2.A, R16.1, U1.K; no longer K11.2, U$2.-VO
- net LIVE_IN: now also R10.2, R12.1, R9.2, T1.A1; no longer K12.P, U$2.AC1
- net LIVE_OUT: now also C4.2, C5.2, T1.A2; no longer K12.S
- net N$4: now also R11.1, U1.T1; no longer K11.1, Q1.E
- net NEUTRAL: now also B1.AC1; no longer U$2.AC2
- net RELAY: now also R13.2; no longer Q1.B
Other:
- moved on the sheet: C2, H1, H2, H3, J1, R5, R6, R7, R8, S1
